File: peripherals_1.sch (KiCad schematic (older format))
At the start: 29 parts, among them J1 Micro_SD_Card_Det, J4 JTAG, J5 Molex_0936263508, J6 USB_A, U1 TXS0108EPW, U6 PCA9546AD, U8 74AC125, U9 TPS2051B

Commit message: cont. work; all connections done now
Parts:
- removed R29, R30, R31: R100, Resistor_SMD:R_0603_1608Metric, symbol trigbox:R100
- removed R32: R100k, Resistor_SMD:R_0603_1608Metric, symbol trigbox:R100k
- added R29, R30, R31: 100, Resistor_SMD:R_0603_1608Metric, symbol Device:R_Small
- added R32: 100k, Resistor_SMD:R_0603_1608Metric, symbol Device:R_Small
- R26, R27: value R100k -> 100k; symbol trigbox:R100k -> Device:R_Small
- R28: value R100 -> 100; symbol trigbox:R100 -> Device:R_Small
- renumbered JP1 to JP3
Changed lines of the file:
@@
 $EndComp
 $Comp
-L trigbox:R100k R26
+L Device:R_Small R26
 U 1 1 5D5F10F0
 P 5550 1350
 F 0 "R26" H 5609 1380 50  0000 L CNN
-F 1 "R100k" V 5550 1350 30  0000 C CNN
+F 1 "100k" V 5550 1350 30  0000 C CNN
 F 2 "Resistor_SMD:R_0603_1608Metric" H 5550 1350 50  0001 C CNN
 F 3 "~" H 5550 1350 50  0001 C CNN
@@
 $EndComp
 $Comp
-L trigbox:R100k R27
+L Device:R_Small R27
 U 1 1 5D5F14E6
 P 5900 1350
 F 0 "R27" H 5959 1380 50  0000 L CNN
-F 1 "R100k" V 5900 1350 30  0000 C CNN
+F 1 "100k" V 5900 1350 30  0000 C CNN
 F 2 "Resistor_SMD:R_0603_1608Metric" H 5900 1350 50  0001 C CNN
 F 3 "~" H 5900 1350 50  0001 C CNN
@@
 Wire Wire Line
 	6500 2000 6850 2000
-$Comp
-L trigbox:R100k R32
-U 1 1 5D5F1573
-P 6850 1900
-F 0 "R32" H 6909 1930 50  0000 L CNN
-F 1 "R100k" V 6850 1900 30  0000 C CNN
-F 2 "Resistor_SMD:R_0603_1608Metric" H 6850 1900 50  0001 C CNN
-F 3 "~" H 6850 1900 50  0001 C CNN
-	1    6850 1900
-	1    0    0    -1
-$EndComp
-$Comp
-L trigbox:R100 R31
-U 1 1 5D5F8A15
-P 6500 1500
-F 0 "R31" H 6500 1350 50  0000 L CNN
-F 1 "R100" V 6500 1500 30  0000 C CNN
-F 2 "Resistor_SMD:R_0603_1608Metric" H 6500 1500 50  0001 C CNN
-F 3 "~" H 6500 1500 50  0001 C CNN
-	1    6500 1500
-	1    0    0    -1
-$EndComp
-$Comp
-L trigbox:R100 R30
-U 1 1 5D5F8E8A
-P 6400 1500
-F 0 "R30" H 6400 1350 50  0000 L CNN
-F 1 "R100" V 6400 1500 30  0000 C CNN
-F 2 "Resistor_SMD:R_0603_1608Metric" H 6400 1500 50  0001 C CNN
-F 3 "~" H 6400 1500 50  0001 C CNN
-	1    6400 1500
-	1    0    0    -1
-$EndComp
-$Comp
-L trigbox:R100 R29
-U 1 1 5D5F8EE0
-P 6300 1500
-F 0 "R29" H 6300 1350 50  0000 L CNN
-F 1 "R100" V 6300 1500 30  0000 C CNN
-F 2 "Resistor_SMD:R_0603_1608Metric" H 6300 1500 50  0001 C CNN
-F 3 "~" H 6300 1500 50  0001 C CNN
-	1    6300 1500
-	1    0    0    -1
-$EndComp
-$Comp
-L trigbox:R100 R28
-U 1 1 5D5F8F38
-P 6200 1500
-F 0 "R28" H 6200 1350 50  0000 L CNN
-F 1 "R100" V 6200 1500 30  0000 C CNN
-F 2 "Resistor_SMD:R_0603_1608Metric" H 6200 1500 50  0001 C CNN
-F 3 "~" H 6200 1500 50  0001 C CNN
-	1    6200 1500
-	1    0    0    -1
-$EndComp
 NoConn ~ 9550 1250
 NoConn ~ 9650 1250
@@
 	3500 3300 3500 3450
 $Comp
-L Device:Jumper_NO_Small JP1
+L Device:Jumper_NO_Small JP3
 U 1 1 60D50F23
 P 3750 2900
-F 0 "JP1" H 3750 2800 50  0000 C CNN
+F 0 "JP3" H 3750 2800 50  0000 C CNN
 F 1 "Jumper_NO_Small" H 3750 2994 50  0000 C CNN
 F 2 "Connector_PinHeader_2.54mm:PinHeader_1x02_P2.54mm_Vertical" H 3750 2900 50  0001 C CNN
@@
 Wire Wire Line
 	2650 4150 3100 4150
+$Comp
+L Device:R_Small R28
+U 1 1 5D5F8F38
+P 6200 1500
+F 0 "R28" V 6150 1250 50  0000 L CNN
+F 1 "100" V 6200 1500 30  0000 C CNN
+F 2 "Resistor_SMD:R_0603_1608Metric" H 6200 1500 50  0001 C CNN
+F 3 "~" H 6200 1500 50  0001 C CNN
+	1    6200 1500
+	1    0    0    -1
+$EndComp
+$Comp
+L Device:R_Small R32
+U 1 1 61011839
+P 6850 1900
+F 0 "R32" H 6909 1930 50  0000 L CNN
+F 1 "100k" V 6850 1900 30  0000 C CNN
+F 2 "Resistor_SMD:R_0603_1608Metric" H 6850 1900 50  0001 C CNN
+F 3 "~" H 6850 1900 50  0001 C CNN
+	1    6850 1900
+	1    0    0    -1
+$EndComp
+$Comp
+L Device:R_Small R29
+U 1 1 61017BC0
+P 6300 1500
+F 0 "R29" V 6250 1250 50  0000 L CNN
+F 1 "100" V 6300 1500 30  0000 C CNN
+F 2 "Resistor_SMD:R_0603_1608Metric" H 6300 1500 50  0001 C CNN
+F 3 "~" H 6300 1500 50  0001 C CNN
+	1    6300 1500
+	1    0    0    -1
+$EndComp
+$Comp
+L Device:R_Small R30
+U 1 1 61017DF1
+P 6400 1500
+F 0 "R30" V 6350 1250 50  0000 L CNN
+F 1 "100" V 6400 1500 30  0000 C CNN
+F 2 "Resistor_SMD:R_0603_1608Metric" H 6400 1500 50  0001 C CNN
+F 3 "~" H 6400 1500 50  0001 C CNN
+	1    6400 1500
+	1    0    0    -1
+$EndComp
+$Comp
+L Device:R_Small R31
+U 1 1 61018026
+P 6500 1500
+F 0 "R31" V 6450 1250 50  0000 L CNN
+F 1 "100" V 6500 1500 30  0000 C CNN
+F 2 "Resistor_SMD:R_0603_1608Metric" H 6500 1500 50  0001 C CNN
+F 3 "~" H 6500 1500 50  0001 C CNN
+	1    6500 1500
+	1    0    0    -1
+$EndComp
 $EndSCHEMATC

Commit message: added more component values/part numbers
Parts:
- FL3: Manufacturer TOKO -> Wurth; Part FDV0530S-1R0 -> 744231371
- J1: Manufacturer (none) -> Hirose; Part (none) -> DM3D-SF
- J5: value Molex_0936263508 -> GigE-RJ45; Manufacturer (none) -> Molex; Part (none) -> 936263508
Changed lines of the file:
@@
 P 9650 2050
 F 0 "J5" V 9183 2050 50  0000 C CNN
-F 1 "Molex_0936263508" V 9274 2050 50  0000 C CNN
+F 1 "GigE-RJ45" V 9274 2050 50  0000 C CNN
 F 2 "proj_footprints:Molex_936263508" H 9650 2050 50  0001 C CNN
 F 3 "" H 9410 1995 50  0001 L TNN
+F 4 "Molex" V 9650 2050 50  0001 C CNN "Manufacturer"
+F 5 "936263508" V 9650 2050 50  0001 C CNN "Part"
 	1    9650 2050
 	-1   0    0    -1
@@
 F 2 "proj_footprints:WE_CNSW" V 9300 6090 50  0001 C CNN
 F 3 "https://www.digikey.com/catalog/en/partgroup/we-cnsw-we-cnsw-hf/22783?mpart=744231371&vendor=732" H 9300 6237 50  0001 C CNN
-F 4 "TOKO" H 9300 6050 50  0001 C CNN "Manufacturer"
-F 5 "FDV0530S-1R0" H 9300 6050 50  0001 C CNN "Part"
+F 4 "Wurth" H 9300 6050 50  0001 C CNN "Manufacturer"
+F 5 "744231371" H 9300 6050 50  0001 C CNN "Part"
 	1    9300 6050
 	1    0    0    1
@@
 F 2 "proj_footprints:microSD_HC_Hirose_DM3D-SF_smaller_crtyd" H 3650 4350 50  0001 C CNN
 F 3 "https://www.hirose.com/product/en/download_file/key_name/DM3/category/Catalog/doc_file_id/49662/?file_category_id=4&item_id=195&is_series=1" H 1600 3750 50  0001 C CNN
+F 4 "DM3D-SF" H 1600 3650 50  0001 C CNN "Part"
+F 5 "Hirose" H 1600 3650 50  0001 C CNN "Manufacturer"
 	1    1600 3650
 	-1   0    0    1

Commit message: re-routed usbA (proper diff-pair); added mounting holes
Connections:
- net labels added: USBA_N, USBA_P
Other:
- moved on the sheet: FL3
Changed lines of the file:
@@
 L fmc:EMI_Filter_LL_14 FL3
 U 1 1 5C29619B
-P 9300 6050
-F 0 "FL3" H 9250 5800 50  0000 C CNN
-F 1 "EMI_Filter_LL_14" H 9300 5600 50  0000 C CNN
-F 2 "proj_footprints:WE_CNSW" V 9300 6090 50  0001 C CNN
-F 3 "https://www.digikey.com/catalog/en/partgroup/we-cnsw-we-cnsw-hf/22783?mpart=744231371&vendor=732" H 9300 6237 50  0001 C CNN
-F 4 "Wurth" H 9300 6050 50  0001 C CNN "Manufacturer"
-F 5 "744231371" H 9300 6050 50  0001 C CNN "Part"
-	1    9300 6050
+P 8550 6050
+F 0 "FL3" H 8500 5800 50  0000 C CNN
+F 1 "EMI_Filter_LL_14" H 8550 5600 50  0000 C CNN
+F 2 "proj_footprints:WE_CNSW" V 8550 6090 50  0001 C CNN
+F 3 "https://www.digikey.com/catalog/en/partgroup/we-cnsw-we-cnsw-hf/22783?mpart=744231371&vendor=732" H 8550 6237 50  0001 C CNN
+F 4 "Wurth" H 8550 6050 50  0001 C CNN "Manufacturer"
+F 5 "744231371" H 8550 6050 50  0001 C CNN "Part"
+	1    8550 6050
 	1    0    0    1
 $EndComp
-Wire Wire Line
-	9500 5950 9500 6000
-Wire Wire Line
-	9500 6000 9800 6000
-Wire Wire Line
-	9500 6150 9500 6100
-Wire Wire Line
-	9500 6100 9800 6100
 $Comp
 L trigbox:R10k R34
@@
 	8850 5750 7400 5750
 Wire Wire Line
-	7400 5950 9100 5950
-Wire Wire Line
-	7400 6150 9100 6150
+	7400 5950 8350 5950
+Wire Wire Line
+	7400 6150 8350 6150
 $Comp
 L power:GND #PWR?
@@
 	1    0    0    -1
 $EndComp
+Wire Wire Line
+	8750 5950 8750 6000
+Wire Wire Line
+	8750 6000 9800 6000
+Wire Wire Line
+	8750 6150 8750 6100
+Wire Wire Line
+	8750 6100 9800 6100
+Text Label 8850 6000 0    50   ~ 0
+USBA_P
+Text Label 8850 6100 0    50   ~ 0
+USBA_N
 $EndSCHEMATC

Commit message: use rj45/Gige + USB combo connector; hooked up LEDs
no more GND window under GigE diff-pairs on power-plane
Parts:
- removed J5: GigE-RJ45, proj_footprints:Molex_936263508, symbol fmc:Molex_0936263508
- removed J6: USB_A, proj_footprints:USB_A_SS52100_001, symbol Connector:USB_A
- added J5: 0821-1X1T-43-F, BEL_0821-1X1T-43-F, symbol fmc:0821-1X1T-43-F
- added R11, R12: 100, Resistor_SMD:R_0603_1608Metric, symbol Device:R_Small
Connections:
- net labels added: B13_L3_N, B13_L3_P, B13_L5_N
- wire segments 177 -> 193
- no-connect marks 10 -> 6
Other:
- moved on the sheet: C1, C12, C14, C15, C3, C4, C5, FL3, J1, J4, JP3, R26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

Commit message: Several changes; converging to prototype version 1.0.0
Added header for connecting external power-supply (in case
chips are not available)
Parts:
- added R13: 10k, Resistor_SMD:R_0603_1608Metric, symbol trigbox:R10k
- C4: value 10uF_1210 -> 10u; footprint Capacitor_SMD:C_1210_3225Metric -> Capacitor_SMD:C_1206_3216Metric; symbol fmc:10uF_1210 -> Device:C; Manufacturer Murata -> Samsung; Part GRJ32ER71E106KE11L -> CL31A106KPHNNNE
- J5: footprint BEL_0821-1X1T-43-F -> proj_footprints:BEL_0821-1X1T-43-F
Connections:
- net +3V3: now also R13.1; no longer U6.3 (RSTb)
- new net B13_L8_N: R13.2, U6.3 (RSTb)
Changed lines of the file:
@@
 Wire Wire Line
 	3550 7150 3550 7600
-$Comp
-L power:+3V3 #PWR?
-U 1 1 5C330733
-P 2750 6700
-AR Path="/5BE73D36/5C330733" Ref="#PWR?"  Part="1"
-AR Path="/5C1147CA/5C330733" Ref="#PWR?"  Part="1"
-F 0 "#PWR?" H 2750 6550 50  0001 C CNN
-F 1 "+3V3" H 2765 6873 50  0000 C CNN
-F 2 "" H 2750 6700 50  0001 C CNN
-F 3 "" H 2750 6700 50  0001 C CNN
-	1    2750 6700
-	1    0    0    -1
-$EndComp
-Wire Wire Line
-	2750 6700 2750 7050
 Wire Wire Line
 	2750 7050 2800 7050
@@
 $EndComp
 $Comp
-L fmc:10uF_1210 C4
+L Device:C C4
 U 1 1 60D50F11
 P 3650 1250
 F 0 "C4" V 3398 1250 50  0000 C CNN
-F 1 "10uF_1210" V 3489 1250 50  0000 C CNN
-F 2 "Capacitor_SMD:C_1210_3225Metric" H 3688 1100 50  0001 C CNN
+F 1 "10u" V 3489 1250 50  0000 C CNN
+F 2 "Capacitor_SMD:C_1206_3216Metric" H 3688 1100 50  0000 C CNN
 F 3 "~" H 3650 1250 50  0001 C CNN
-F 4 "GRJ32ER71E106KE11L" H 3775 1450 50  0001 C CNN "Part"
-F 5 "Murata" H 3875 1550 50  0001 C CNN "Manufacturer"
+F 4 "CL31A106KPHNNNE" H 3775 1450 50  0001 C CNN "Part"
+F 5 "Samsung" H 3875 1550 50  0001 C CNN "Manufacturer"
 	1    3650 1250
 	0    1    1    0
 $EndComp
-Connection ~ 3800 1250
 Wire Wire Line
 	3500 1250 3300 1250
@@
 F 0 "J5" H 9750 5267 50  0000 C CNN
 F 1 "0821-1X1T-43-F" H 9750 5176 50  0000 C CNN
-F 2 "BEL_0821-1X1T-43-F" H 9800 3600 50  0001 L BNN
+F 2 "proj_footprints:BEL_0821-1X1T-43-F" H 9800 3600 50  0001 L BNN
 F 3 "https://www.digikey.com/product-detail/en/bel-fuse-inc/0821-1X1T-43-F/507-1567-ND/2257870?utm_source=snapeda&utm_medium=aggregator&utm_campaign=symbol" H 9800 3600 50  0001 L BNN
 F 4 "507-1567-ND" H 9800 3600 50  0001 L BNN "Field4"
@@
 Text GLabel 8350 4900 0    50   Input ~ 0
 B13_L5_N
+$Comp
+L power:+3V3 #PWR?
+U 1 1 5C330733
+P 2750 6350
+AR Path="/5BE73D36/5C330733" Ref="#PWR?"  Part="1"
+AR Path="/5C1147CA/5C330733" Ref="#PWR?"  Part="1"
+F 0 "#PWR?" H 2750 6200 50  0001 C CNN
+F 1 "+3V3" H 2765 6523 50  0000 C CNN
+F 2 "" H 2750 6350 50  0001 C CNN
+F 3 "" H 2750 6350 50  0001 C CNN
+	1    2750 6350
+	1    0    0    -1
+$EndComp
+Text GLabel 1800 7050 0    50   Input ~ 0
+B13_L8_N
+Wire Wire Line
+	1800 7050 2750 7050
+Connection ~ 2750 7050
+$Comp
+L trigbox:R10k R?
+U 1 1 60F55A10
+P 2750 6450
+AR Path="/60DAA393/5C4CE703/60F55A10" Ref="R?"  Part="1"
+AR Path="/5C1147CA/60F55A10" Ref="R13"  Part="1"
+F 0 "R13" H 2809 6480 50  0000 L CNN
+F 1 "10k" H 2809 6404 30  0000 L CNN
+F 2 "Resistor_SMD:R_0603_1608Metric" H 2750 6450 50  0001 C CNN
+F 3 "~" H 2750 6450 50  0001 C CNN
+	1    2750 6450
+	-1   0    0    -1
+$EndComp
+Wire Wire Line
+	2750 6550 2750 7050
 $EndSCHEMATC

Commit message: WIP: (save)
Parts:
- removed C12, C13, C2, C3, C5: 100nF_603, Capacitor_SMD:C_0603_1608Metric, symbol fmc:100nF_603
- removed C14, C15: 47uF, 10V, Capacitor_SMD:C_1206_3216Metric, symbol Device:CP1_Small
- removed C4: 10u, Capacitor_SMD:C_1206_3216Metric, symbol Device:C
- removed FL3: EMI_Filter_LL_14, proj_footprints:WE_CNSW, symbol fmc:EMI_Filter_LL_14
- removed J1: Micro_SD_Card_Det, proj_footprints:microSD_HC_Hirose_DM3D-SF_smaller_crtyd, symbol Connector:Micro_SD_Card_Det
- removed J5: 0821-1X1T-43-F, proj_footprints:BEL_0821-1X1T-43-F, symbol fmc:0821-1X1T-43-F
- removed JP3: Jumper_NO_Small, Connector_PinHeader_2.54mm:PinHeader_1x02_P2.54mm_Vertical, symbol Device:Jumper_NO_Small
- removed R11, R12: 100, Resistor_SMD:R_0603_1608Metric, symbol Device:R_Small
- removed R13, R34: 10k, Resistor_SMD:R_0603_1608Metric, symbol trigbox:R10k
- removed RN1, RN2: 4x4k7, Resistor_SMD:R_Array_Convex_4x0603, symbol Device:R_Pack04
- removed U1: TXS0108EPW, Package_SO:TSSOP-20_4.4x6.5mm_P0.65mm, symbol Logic_LevelTranslator:TXS0108EPW
- removed U6: PCA9546AD, Package_SO:SOIC-16_3.9x9.9mm_P1.27mm, symbol fmc:PCA9546AD
- removed U9: TPS2051B, Package_TO_SOT_SMD:SOT-23-5, symbol fmc:TPS2051B
- added C34, C35: 47p, Capacitor_SMD:C_0603_1608Metric, symbol Device:C_Small
- added C36, C38, C39: 100n, Capacitor_SMD:C_0603_1608Metric, symbol fmc:100nF_603
- added C37: 10u, Capacitor_SMD:C_1206_3216Metric, symbol Device:C_Small
- added D1, D2, D3, D4, D5, D6, D7, D8: LED, LED_SMD:LED_0603_1608Metric, symbol Device:LED
- added R10, R3, R4, R5, R6, R7, R8, R9: 1k, Resistor_SMD:R_0603_1608Metric, symbol Device:R_Small
- added R19: 0, Resistor_SMD:R_0402_1005Metric, symbol Device:R_Small
- added R20, R21: 27, Resistor_SMD:R_0603_1608Metric, symbol Device:R_Small
- added U3: FT240XQ, Package_DFN_QFN:QFN-24-1EP_4x4mm_P0.5mm_EP2.6x2.6mm, symbol fmc:FT240XQ
- U8: value 74AC125 -> 74ALVC125
Connections:
- net +3V3 is gone; now on net +1V8: C1.2, R26.1, R27.1, R32.1, U8.14 (Vcc)
- net VREF_JTAG is gone; now on net +1V8: J4.6 (Pin_6)
- net +1V8: now also C39.2, U3.24 (VCCIO)
- net +5V: now also C37.1, C38.2, U3.15 (VCC)
- net GND: now also C34.1, C35.2, C36.1, C37.2, C38.1, C39.1, D1.1 (K), D2.1 (K), D3.1 (K), D4.1 (K), D5.1 (K), D6.1 (K), D7.1 (K), D8.1 (K), U3.16 (GND), U3.25 (GND), U3.3 (GND)
- new net: C36.2, U3.12 (3V3OUT), U3.13 (~RESET)
- new net: D1.2 (A), R3.2
- new net: D2.2 (A), R4.2
- new net: D3.2 (A), R5.2
- new net: D4.2 (A), R6.2
- new net: D5.2 (A), R7.2
- new net: D6.2 (A), R8.2
- new net: D7.2 (A), R9.2
- new net: D8.2 (A), R10.2
- new net B13_L15_N: R3.1
- new net B13_L15_P: R4.1
- new net B13_L18_N: R9.1
- new net B13_L18_P: R10.1
- new net B13_L20_N: R6.1
- new net B13_L20_P: R5.1
- new net B13_L21_N: R8.1
- new net B13_L21_P: R7.1
- new net FIFO_CLK: R19.1, U3.19 (CBUS6)
- new net FIFO_D0: U3.21 (DATA0)
- new net FIFO_D1: U3.1 (DATA1)
- new net FIFO_D2: U3.23 (DATA2)
- new net FIFO_D3: U3.6 (DATA3)
- new net FIFO_D4: U3.22 (DATA4)
- new net FIFO_D5: U3.4 (DATA5)
- new net FIFO_D6: U3.5 (DATA6)
- new net FIFO_D7: U3.2 (DATA7)
- new net FIFO_RDb: U3.8 (~RD)
- new net FIFO_RXE: U3.18 (~RXF)
- new net FIFO_SIWU: U3.7 (~SI/WU)
- new net FIFO_TXF: U3.17 (~TXE)
- new net FIFO_WRb: U3.9 (~WR)
- new net USBD_N: R21.2, U3.11 (USBDM)
- new net USBD_P: R20.2, U3.10 (USBDP)
- new net USB_BCDb: R19.2
- new net USB_PWRENb: U3.20 (CBUS5)
- new net USBin_N: C35.1, R21.1
- new net USBin_P: C34.2, R20.1
- no-connect marks 6 -> 1
Other:
- note added: "GREEN LED"
- note added: "RED LED"
- note removed: "PGOOD is 3v3 but OE is\nreferenced to VCCA"
- note removed: "Write-protect"
- moved on the sheet: J4, R32

Commit message: WIP: point before we change to OSH/relaxed process
Parts:
- added Q1: SSM6N35AFE, proj_footprints:SOT-563-adjusted, symbol Device:Q_DUAL_NMOS_S1G1D2S2G2D1
- added R2, R72: 3k3, Resistor_SMD:R_0603_1608Metric, symbol Device:R_Small
- added R73, R74: 10k, Resistor_SMD:R_0603_1608Metric, symbol Device:R_Small
Connections:
- net B13_L15_N renamed LED1
- net B13_L15_P renamed LED2
- net B13_L18_N renamed LED7
- net B13_L18_P renamed LED8
- net B13_L20_N renamed LED4
- net B13_L20_P renamed LED3
- net B13_L21_N renamed LED6
- net B13_L21_P renamed LED5
- new net +1V8_lan9254: Q1.2 (G), Q1.5 (G), R2.1, R72.1
- new net +3V3: R73.1, R74.1
- new net SCL0: R72.2
- new net SCL1_3V3: Q1.6 (D), R73.2
- new net SCL_1: Q1.1 (S)
- new net SDA0: R2.2
- new net SDA1_3V3: Q1.3 (D), R74.2
- new net SDA_1: Q1.4 (S)
Other:
- note added: "FIXME -- LEDs need driver (3v3 or 5v) !!"
- moved on the sheet: C1, J4, R26, R27, R28, R29, R30, R31, R32, U8
