File: peripherals_1.sch (KiCad schematic (older format))
At the start: 41 parts, among them J4 JTAG, Q1 SSM6N35AFE, U3 FT240XQ, U8 74ALVC125

Commit message: re-routed with more relaxed specs (that eurocircuits can also meet)
No chance with OSH, however...

Going to place stuff on the board now...
Parts:
- R19: footprint Resistor_SMD:R_0402_1005Metric -> Resistor_SMD:R_0603_1608Metric
Changed lines of the file:
@@
 F 0 "R19" V 5800 3150 50  0000 C CNN
 F 1 "0" V 5700 3150 50  0000 C CNN
-F 2 "Resistor_SMD:R_0402_1005Metric" H 5550 3150 50  0001 C CNN
+F 2 "Resistor_SMD:R_0603_1608Metric" H 5550 3150 50  0001 C CNN
 F 3 "~" H 5550 3150 50  0001 C CNN
 	1    5550 3150

Commit message: further work...
Parts:
- removed D1, D2, D3, D4, D5, D6, D7, D8: LED, LED_SMD:LED_0603_1608Metric, symbol Device:LED
- removed R10, R3, R4, R5, R6, R7, R8, R9: 1k, Resistor_SMD:R_0603_1608Metric, symbol Device:R_Small
- added R83: 100k, Resistor_SMD:R_0603_1608Metric, symbol Device:R_Small
- U8: footprint Package_SO:SOIC-14_3.9x8.7mm_P1.27mm -> Package_SO:TSSOP-14_4.4x5mm_P0.65mm
Connections:
- net +1V8: now also R83.1
- net GND: no longer U8.13 (OE2b)
- net TCK: now also U8.6 (Y1); no longer U8.3 (Y0)
- net TCK_I: now also U8.5 (X1); no longer U8.2 (X0)
- net TDI: now also U8.8 (Y3); no longer U8.6 (Y1)
- net TDI_I: now also U8.9 (X3); no longer U8.5 (X1)
- net TDO: now also R83.2
- net TMS: now also U8.3 (Y0); no longer U8.8 (Y3)
- net TMS_I: now also U8.2 (X0); no longer U8.9 (X3)
- new net TDO_OEb: U8.13 (OE2b)
Other:
- note added: "This driver is just for protection\nisolating the FPGA pins.\nIt also muxes the TDO signal."
- note removed: "FIXME -- LEDs need driver (3v3 or 5v) !!"
- note removed: "GREEN LED"
- note removed: "RED LED"
- moved on the sheet: C1, C34, C35, C36, C37, C38, C39, R19, R20, R21, U3
