File: fpga_bank0_cfg.sch (KiCad schematic (older format))
At the start: 10 parts, among them SW1 PROG, U1 XC7A35T-CSG325

Commit message: WIP: point before we change to OSH/relaxed process
Parts:
- removed R2: 50, Resistor_SMD:R_0603_1608Metric, symbol Device:R_Small
- U1: symbol FPGA_Xilinx_Artix7:XC7A35T-CSG325 -> fmc:XC7A35T-CSG325
Connections:
- wire segments 50 -> 49
Changed lines of the file:
@@
 $Descr A4 11693 8268
 encoding utf-8
-Sheet 11 18
+Sheet 10 18
 Title ""
 Date ""
@@
 $EndDescr
 $Comp
-L FPGA_Xilinx_Artix7:XC7A35T-CSG325 U1
+L fmc:XC7A35T-CSG325 U1
 U 5 1 62263CAE
 P 2700 3000
@@
 Wire Wire Line
 	4200 4000 4200 4100
-$Comp
-L Device:R_Small R2
-U 1 1 622E8D22
-P 4450 2700
-AR Path="/620D1E32/622637A6/622E8D22" Ref="R2"  Part="1"
-AR Path="/620D1E32/622D3D90/622E8D22" Ref="R?"  Part="1"
-F 0 "R2" V 4400 2850 50  0000 C CNN
-F 1 "50" V 4400 3150 50  0000 C CNN
-F 2 "Resistor_SMD:R_0603_1608Metric" H 4450 2700 50  0001 C CNN
-F 3 "~" H 4450 2700 50  0001 C CNN
-	1    4450 2700
-	0    1    1    0
-$EndComp
 Text HLabel 5050 2700 2    50   Output ~ 0
 CCLK
-Wire Wire Line
-	4200 2700 4350 2700
-Wire Wire Line
-	4550 2700 5050 2700
 Wire Wire Line
 	4200 2900 4750 2900
@@
 Wire Wire Line
 	5600 3200 5600 2950
+Wire Wire Line
+	4200 2700 5050 2700
 $EndSCHEMATC

Commit message: further work...
Parts:
- removed R63: 4k7, Resistor_SMD:R_0603_1608Metric, symbol Device:R_Small
- removed SW1: PROG, Button_Switch_SMD:SW_SPST_PTS810, symbol Switch:SW_Push
- added R84: 4k7, Resistor_SMD:R_0603_1608Metric, symbol Device:R_Small
- added SW1: PROG, proj_footprints:SW_SPST_PTS810_and_PTS841, symbol fmc:SW_Push_Shielded
Connections:
- net +1V8: now also R84.2
- net GND: now also SW1.1, SW1.3 (Shield)
- net DONE: now reaches U1.F12 (DONE_0)
- net DONE: now also R84.1
- net at R12.1, U1.P10 (PROGRAM_B_0): now also SW1.2
Changed lines of the file:
@@
 $Descr A4 11693 8268
 encoding utf-8
-Sheet 10 18
+Sheet 5 20
 Title ""
 Date ""
@@
 Wire Wire Line
 	5850 3400 5850 2950
-$Comp
-L Switch:SW_Push SW1
-U 1 1 6231C540
-P 5150 3600
-F 0 "SW1" H 5150 3800 50  0000 C CNN
-F 1 "PROG" H 4950 3700 50  0000 C CNN
-F 2 "Button_Switch_SMD:SW_SPST_PTS810" H 5150 3800 50  0001 C CNN
-F 3 "~" H 5150 3800 50  0001 C CNN
-	1    5150 3600
-	-1   0    0    1
-$EndComp
 Wire Wire Line
 	4950 3600 4750 3600
@@
 L power:GND #PWR?
 U 1 1 62324145
-P 5750 3600
+P 5750 3850
 AR Path="/5C114F28/5C114F4B/62324145" Ref="#PWR?"  Part="1"
 AR Path="/5C114F28/5C1157BA/62324145" Ref="#PWR?"  Part="1"
@@
 AR Path="/620D1E32/620D23E9/62324145" Ref="#PWR?"  Part="1"
 AR Path="/620D1E32/622637A6/62324145" Ref="#PWR?"  Part="1"
-F 0 "#PWR?" H 5750 3350 50  0001 C CNN
-F 1 "GND" H 5755 3427 50  0000 C CNN
-F 2 "" H 5750 3600 50  0001 C CNN
-F 3 "" H 5750 3600 50  0001 C CNN
-	1    5750 3600
-	1    0    0    -1
-$EndComp
+F 0 "#PWR?" H 5750 3600 50  0001 C CNN
+F 1 "GND" H 5755 3677 50  0000 C CNN
+F 2 "" H 5750 3850 50  0001 C CNN
+F 3 "" H 5750 3850 50  0001 C CNN
+	1    5750 3850
+	1    0    0    -1
+$EndComp
+Wire Wire Line
+	4200 2700 5050 2700
+Wire Wire Line
+	4200 3200 6500 3200
+Connection ~ 6150 2650
+$Comp
+L fmc:SW_Push_Shielded SW1
+U 1 1 6258B48E
+P 5150 3600
+F 0 "SW1" H 5500 3700 50  0000 C CNN
+F 1 "PROG" H 4950 3700 50  0000 C CNN
+F 2 "proj_footprints:SW_SPST_PTS810_and_PTS841" H 5150 3800 50  0001 C CNN
+F 3 "~" H 5150 3800 50  0001 C CNN
+	1    5150 3600
+	1    0    0    -1
+$EndComp
+Wire Wire Line
+	5150 3850 5750 3850
+Wire Wire Line
+	5750 3850 5750 3600
 Wire Wire Line
 	5750 3600 5900 3600
-$Comp
-L Device:R_Small R63
-U 1 1 6243709B
-P 5600 2850
-AR Path="/620D1E32/622637A6/6243709B" Ref="R63"  Part="1"
-AR Path="/620D1E32/622D3D90/6243709B" Ref="R?"  Part="1"
-F 0 "R63" H 5500 2800 50  0000 C CNN
-F 1 "4k7" H 5500 2900 50  0000 C CNN
-F 2 "Resistor_SMD:R_0603_1608Metric" H 5600 2850 50  0001 C CNN
-F 3 "~" H 5600 2850 50  0001 C CNN
-	1    5600 2850
+Connection ~ 5750 3850
+$Comp
+L Device:R_Small R84
+U 1 1 625DF7BB
+P 6500 2850
+AR Path="/620D1E32/622637A6/625DF7BB" Ref="R84"  Part="1"
+AR Path="/620D1E32/622D3D90/625DF7BB" Ref="R?"  Part="1"
+F 0 "R84" H 6400 2800 50  0000 C CNN
+F 1 "4k7" H 6400 2900 50  0000 C CNN
+F 2 "Resistor_SMD:R_0603_1608Metric" H 6500 2850 50  0001 C CNN
+F 3 "~" H 6500 2850 50  0001 C CNN
+	1    6500 2850
 	-1   0    0    1
 $EndComp
 Wire Wire Line
-	5600 2750 5600 2650
-Wire Wire Line
-	5600 2650 5850 2650
-Wire Wire Line
-	4200 3200 5600 3200
-Wire Wire Line
-	5600 3200 5600 2950
-Wire Wire Line
-	4200 2700 5050 2700
+	6500 2750 6500 2650
+Wire Wire Line
+	6500 2650 6150 2650
+Wire Wire Line
+	6500 2950 6500 3200
+Text HLabel 6800 3200 2    50   Output ~ 0
+DONE
+Wire Wire Line
+	6500 3200 6800 3200
+Connection ~ 6500 3200
+Text HLabel 6800 2650 2    50   Output ~ 0
+VCCO_0
+Wire Wire Line
+	6500 2650 6800 2650
+Connection ~ 6500 2650
 $EndSCHEMATC
