File: fpga_bank14_15.sch (KiCad schematic (older format))
At the start: 22 parts, among them U1 XC7A35T-CSG325, U2 AT25SL641

Commit message: WIP: point before we change to OSH/relaxed process
Parts:
- added C86: 100n, Capacitor_SMD:C_0603_1608Metric, symbol Device:C_Small
- U1: symbol FPGA_Xilinx_Artix7:XC7A35T-CSG325 -> fmc:XC7A35T-CSG325
Connections:
- wire segments 78 -> 79
Changed lines of the file:
@@
 $Descr A4 11693 8268
 encoding utf-8
-Sheet 13 18
+Sheet 7 18
 Title ""
 Date ""
@@
 $EndDescr
 $Comp
-L FPGA_Xilinx_Artix7:XC7A35T-CSG325 U1
+L fmc:XC7A35T-CSG325 U1
 U 1 1 622D4082
 P 4150 4050
@@
 	-1   0    0    -1
 $EndComp
+$Comp
+L Device:C_Small C86
+U 1 1 621FD204
+P 9550 2550
+F 0 "C86" H 9642 2596 50  0000 L CNN
+F 1 "100n" H 9642 2505 50  0000 L CNN
+F 2 "Capacitor_SMD:C_0603_1608Metric" H 9550 2550 50  0001 C CNN
+F 3 "~" H 9550 2550 50  0001 C CNN
+	1    9550 2550
+	1    0    0    -1
+$EndComp
+$Comp
+L power:GND #PWR?
+U 1 1 621FD7D4
+P 9550 2650
+AR Path="/5C114F28/5C114F4B/621FD7D4" Ref="#PWR?"  Part="1"
+AR Path="/5C114F28/5C1157BA/621FD7D4" Ref="#PWR?"  Part="1"
+AR Path="/5C439C1E/621FD7D4" Ref="#PWR?"  Part="1"
+AR Path="/5C439C2E/621FD7D4" Ref="#PWR?"  Part="1"
+AR Path="/5C439C1E/5C801264/621FD7D4" Ref="#PWR?"  Part="1"
+AR Path="/5C439C1E/5C83CE66/621FD7D4" Ref="#PWR?"  Part="1"
+AR Path="/5C439C2E/5C801264/621FD7D4" Ref="#PWR?"  Part="1"
+AR Path="/5C439C2E/5C83CE66/621FD7D4" Ref="#PWR?"  Part="1"
+AR Path="/5C439C1E/5C847C02/621FD7D4" Ref="#PWR?"  Part="1"
+AR Path="/5C439C2E/5C847C02/621FD7D4" Ref="#PWR?"  Part="1"
+AR Path="/621FD7D4" Ref="#PWR?"  Part="1"
+AR Path="/620D1E32/620D23E9/621FD7D4" Ref="#PWR?"  Part="1"
+AR Path="/620D1E32/622637A6/621FD7D4" Ref="#PWR?"  Part="1"
+AR Path="/620D1E32/622D3D90/621FD7D4" Ref="#PWR?"  Part="1"
+F 0 "#PWR?" H 9550 2400 50  0001 C CNN
+F 1 "GND" H 9555 2477 50  0000 C CNN
+F 2 "" H 9550 2650 50  0001 C CNN
+F 3 "" H 9550 2650 50  0001 C CNN
+	1    9550 2650
+	1    0    0    -1
+$EndComp
+Wire Wire Line
+	9550 2450 9150 2450
 $EndSCHEMATC

Commit message: further work...
Parts:
- added R82: 100k, Resistor_SMD:R_0603_1608Metric, symbol Device:R_Small
- R15, R16, R17: value 2k4 -> 10k
Connections:
- net +1V8: now also R82.1
- net at U1.K16 (IO_L1P_T0_D00_MOSI_14), U2.5 (SI/SIO0): now also R82.2
Changed lines of the file:
@@
 $Descr A4 11693 8268
 encoding utf-8
-Sheet 7 18
+Sheet 7 20
 Title ""
 Date ""
@@
 	1    0    0    -1
 $EndComp
-Text Notes 8300 2050 0    50   ~ 0
+Text Notes 8300 1700 0    50   ~ 0
 64Mbit, 1.8V, must be ready < TPOR = 10ms
 $Comp
@@
 L power:+1V8 #PWR?
 U 1 1 622E031F
-P 9150 2400
+P 9150 1950
 AR Path="/5C0C1285/622E031F" Ref="#PWR?"  Part="1"
 AR Path="/5C114F28/5C114F49/622E031F" Ref="#PWR?"  Part="1"
@@
 AR Path="/620D1E32/622637A6/622E031F" Ref="#PWR?"  Part="1"
 AR Path="/620D1E32/622D3D90/622E031F" Ref="#PWR?"  Part="1"
-F 0 "#PWR?" H 9150 2250 50  0001 C CNN
-F 1 "+1V8" H 9165 2573 50  0000 C CNN
-F 2 "" H 9150 2400 50  0001 C CNN
-F 3 "" H 9150 2400 50  0001 C CNN
-	1    9150 2400
+F 0 "#PWR?" H 9150 1800 50  0001 C CNN
+F 1 "+1V8" H 9165 2123 50  0000 C CNN
+F 2 "" H 9150 1950 50  0001 C CNN
+F 3 "" H 9150 1950 50  0001 C CNN
+	1    9150 1950
 	1    0    0    -1
 $EndComp
@@
 AR Path="/620D1E32/622D3D90/622E0325" Ref="R17"  Part="1"
 F 0 "R17" V 8350 2900 50  0000 C CNN
-F 1 "2k4" V 8350 3200 50  0000 C CNN
+F 1 "10k" V 8350 3200 50  0000 C CNN
 F 2 "Resistor_SMD:R_0603_1608Metric" H 8400 2750 50  0001 C CNN
 F 3 "~" H 8400 2750 50  0001 C CNN
@@
 	8500 2750 9150 2750
 Wire Wire Line
-	9150 2400 9150 2450
+	9150 1950 9150 2300
 Wire Wire Line
 	8450 3350 8250 3350
@@
 AR Path="/620D1E32/622D3D90/622E0332" Ref="R16"  Part="1"
 F 0 "R16" V 8350 2750 50  0000 C CNN
-F 1 "2k4" V 8350 3050 50  0000 C CNN
+F 1 "10k" V 8350 3050 50  0000 C CNN
 F 2 "Resistor_SMD:R_0603_1608Metric" H 8400 2600 50  0001 C CNN
 F 3 "~" H 8400 2600 50  0001 C CNN
@@
 AR Path="/620D1E32/622D3D90/622E0338" Ref="R15"  Part="1"
 F 0 "R15" V 8350 2600 50  0000 C CNN
-F 1 "2k4" V 8350 2900 50  0000 C CNN
+F 1 "10k" V 8350 2900 50  0000 C CNN
 F 2 "Resistor_SMD:R_0603_1608Metric" H 8400 2450 50  0001 C CNN
 F 3 "~" H 8400 2450 50  0001 C CNN
@@
 	8050 3550 8450 3550
 Wire Wire Line
-	7850 2050 7850 3150
+	7850 2050 7850 2300
 Wire Wire Line
 	7850 3150 8450 3150
@@
 Wire Wire Line
 	9550 2450 9150 2450
+$Comp
+L Device:R_Small R?
+U 1 1 626A7F0C
+P 8400 2300
+AR Path="/620D1E32/622637A6/626A7F0C" Ref="R?"  Part="1"
+AR Path="/620D1E32/622D3D90/626A7F0C" Ref="R82"  Part="1"
+F 0 "R82" V 8350 2450 50  0000 C CNN
+F 1 "100k" V 8350 2750 50  0000 C CNN
+F 2 "Resistor_SMD:R_0603_1608Metric" H 8400 2300 50  0001 C CNN
+F 3 "~" H 8400 2300 50  0001 C CNN
+	1    8400 2300
+	0    1    1    0
+$EndComp
+Wire Wire Line
+	7850 2300 8300 2300
+Connection ~ 7850 2300
+Wire Wire Line
+	7850 2300 7850 3150
+Wire Wire Line
+	8500 2300 9150 2300
+Connection ~ 9150 2300
+Wire Wire Line
+	9150 2300 9150 2450
 $EndSCHEMATC
