File: fpga_gtp.sch (KiCad schematic (older format))
At the start: 1 part, among them U1 XC7A35T-CSG325

Commit message: WIP: point before we change to OSH/relaxed process
Parts:
- U1: symbol FPGA_Xilinx_Artix7:XC7A35T-CSG325 -> fmc:XC7A35T-CSG325
Changed lines of the file:
@@
 $Descr A4 11693 8268
 encoding utf-8
-Sheet 12 18
+Sheet 11 18
 Title ""
 Date ""
@@
 $EndDescr
 $Comp
-L FPGA_Xilinx_Artix7:XC7A35T-CSG325 U1
+L fmc:XC7A35T-CSG325 U1
 U 3 1 622B68F5
 P 7150 3200
