File: sfp-conn.sch (KiCad schematic (older format))
At the start: 10 parts, among them J19 SFP, J20 SFP_CAGE

Commit message: Several changes; converging to prototype version 1.0.0
Added header for connecting external power-supply (in case
chips are not available)
Parts:
- C57, C60: value 10uF_1210 -> 10u; footprint Capacitor_SMD:C_1210_3225Metric -> Capacitor_SMD:C_1206_3216Metric; symbol fmc:10uF_1210 -> Device:C; Manufacturer Murata -> Samsung; Part GRJ32ER71E106KE11L -> CL31A106KPHNNNE
Changed lines of the file:
@@
 $EndComp
 $Comp
-L fmc:10uF_1210 C?
+L Device:C C?
 U 1 1 5BDFCC25
 P 2300 2850
@@
 AR Path="/5C210D20/5BDFCC25" Ref="C69"  Part="1"
 F 0 "C57" H 2415 2896 50  0000 L CNN
-F 1 "10uF_1210" H 2415 2805 50  0000 L CNN
-F 2 "Capacitor_SMD:C_1210_3225Metric" H 2338 2700 50  0001 C CNN
+F 1 "10u" H 2415 2805 50  0000 L CNN
+F 2 "Capacitor_SMD:C_1206_3216Metric" H 2338 2700 50  0001 C CNN
 F 3 "~" H 2300 2850 50  0001 C CNN
-F 4 "Murata" H 0   0   50  0001 C CNN "Manufacturer"
-F 5 "GRJ32ER71E106KE11L" H 0   0   50  0001 C CNN "Part"
+F 4 "Samsung" H 0   0   50  0001 C CNN "Manufacturer"
+F 5 "CL31A106KPHNNNE" H 0   0   50  0001 C CNN "Part"
 	1    2300 2850
 	-1   0    0    -1
@@
 $EndComp
 $Comp
-L fmc:10uF_1210 C?
+L Device:C C?
 U 1 1 5BDFCC5D
 P 4350 2850
@@
 AR Path="/5C210D20/5BDFCC5D" Ref="C72"  Part="1"
 F 0 "C60" H 4465 2896 50  0000 L CNN
-F 1 "10uF_1210" H 4465 2805 50  0000 L CNN
-F 2 "Capacitor_SMD:C_1210_3225Metric" H 4388 2700 50  0001 C CNN
+F 1 "10u" H 4465 2805 50  0000 L CNN
+F 2 "Capacitor_SMD:C_1206_3216Metric" H 4388 2700 50  0001 C CNN
 F 3 "~" H 4350 2850 50  0001 C CNN
-F 4 "Murata" H 0   0   50  0001 C CNN "Manufacturer"
-F 5 "GRJ32ER71E106KE11L" H 0   0   50  0001 C CNN "Part"
+F 4 "Samsung" H 0   0   50  0001 C CNN "Manufacturer"
+F 5 "CL31A106KPHNNNE" H 0   0   50  0001 C CNN "Part"
 	1    4350 2850
 	1    0    0    -1

Commit message: WIP: (save)
Connections:
- net SFP_RX_N: now also J19.12 (RD-); no longer J19.13 (RD+)
- net SFP_RX_P: now also J19.13 (RD+); no longer J19.12 (RD-)
Changed lines of the file:
@@
 $Descr USLetter 11000 8500
 encoding utf-8
-Sheet 4 12
+Sheet 3 18
 Title "Timing FMC"
 Date "2018-11-01"
@@
 	3200 2700 2900 2700
 Connection ~ 2550 2700
-Text HLabel 3350 4300 0    50   Output ~ 0
+Text HLabel 3350 4400 0    50   Output ~ 0
 SFP_RX_P
 Text HLabel 3350 4550 0    50   Input ~ 0
@@
 Connection ~ 5550 5400
 Connection ~ 5450 5400
-Text HLabel 3350 4400 0    50   Output ~ 0
+Text HLabel 3350 4300 0    50   Output ~ 0
 SFP_RX_N
 Text HLabel 8350 4600 2    50   Output ~ 0

Commit message: further work...
Parts:
- added R85, R88, R91: 4k7, Resistor_SMD:R_0603_1608Metric, symbol Device:R_Small
- added R92, R93, R94, R95, R96, R97: 47k, Resistor_SMD:R_0603_1608Metric, symbol Device:R_Small
Connections:
- net +3V3: now also R85.2, R88.2, R91.2
- net GND: now also R93.1, R95.1, R97.1
- net LOS: now also R94.1, R95.2; no longer J19.8 (LOS)
- net PRESENTb: now also R92.1, R93.2; no longer J19.6 (MOD_DEF0/PRESENTb)
- net TX_FAULT: now also R96.1, R97.2; no longer J19.2 (TX_FAULT)
- new net: J19.2 (TX_FAULT), R85.1, R96.2
- new net: J19.6 (MOD_DEF0/PRESENTb), R91.1, R92.2
- new net: J19.8 (LOS), R88.1, R94.2
Other:
- note added: "Resistor values shown for level conversion to 1.8V"
- note removed: "Note: enable pull-ups on FPGA inputs\nfor LOS, TX_FAULT, PRESENTb"
