File: fpga_power.sch (KiCad schematic (older format))
At the start: 28 parts, among them U1 XC7A35T-CSG325

Commit message: WIP: point before we change to OSH/relaxed process
Parts:
- U1: symbol FPGA_Xilinx_Artix7:XC7A35T-CSG325 -> fmc:XC7A35T-CSG325
Changed lines of the file:
@@
 $Descr A4 11693 8268
 encoding utf-8
-Sheet 10 18
+Sheet 4 18
 Title ""
 Date ""
@@
 $EndDescr
 $Comp
-L FPGA_Xilinx_Artix7:XC7A35T-CSG325 U1
+L fmc:XC7A35T-CSG325 U1
 U 6 1 620D2B05
 P 3250 4000
@@
 $EndComp
 $Comp
-L FPGA_Xilinx_Artix7:XC7A35T-CSG325 U1
+L fmc:XC7A35T-CSG325 U1
 U 4 1 620DFECC
 P 7250 5100

Commit message: further work...
Parts:
- C22: footprint Capacitor_SMD:C_0603_1608Metric -> Capacitor_SMD:C_0402_1005Metric
Changed lines of the file:
@@
 $Descr A4 11693 8268
 encoding utf-8
-Sheet 4 18
+Sheet 4 20
 Title ""
 Date ""
@@
 F 0 "C22" H 8842 1146 50  0000 L CNN
 F 1 "470n" H 8842 1055 50  0000 L CNN
-F 2 "Capacitor_SMD:C_0603_1608Metric" H 8750 1100 50  0001 C CNN
+F 2 "Capacitor_SMD:C_0402_1005Metric" H 8750 1100 50  0001 C CNN
 F 3 "~" H 8750 1100 50  0001 C CNN
 	1    8750 1100

Commit message: updated cap footprint
Parts:
- C21: footprint proj_footprints:C_pol_1210_3225Metric -> Capacitor_Tantalum_SMD:CP_EIA-3528-15_AVX-H
Changed lines of the file:
@@
 F 0 "C21" H 8441 1146 50  0000 L CNN
 F 1 "100u" H 8441 1055 50  0000 L CNN
-F 2 "proj_footprints:C_pol_1210_3225Metric" H 8350 1100 50  0001 C CNN
+F 2 "Capacitor_Tantalum_SMD:CP_EIA-3528-15_AVX-H" H 8350 1100 50  0001 C CNN
 F 3 "~" H 8350 1100 50  0001 C CNN
 	1    8350 1100
