File: kicad/ecevr-proto.kicad_sch (KiCad schematic)
At the start: 5 parts, among them U21 74LVC1G06

Commit message: WIP
Connections:
- net IO_L3N_T0_DQS_AD1N_15: no longer names the net of U21.1, U21.2
Other:
- removed sheet fpga
- removed sheet pof_io
- added sheet b2b_conn (te0714_b2b.kicad_sch)
- sheet USB, JTAG, I2C ports: added VREF_JTAG; removed FIFO_CBUS5, FIFO_CLK, FIFO_D0, FIFO_D1, FIFO_D2, FIFO_D3, FIFO_D4, FIFO_D5, FIFO_D6, FIFO_D7, FIFO_RDb, FIFO_RXE, FIFO_SIWU, FIFO_TXF, FIFO_WRb
- sheet lan9254 ports: added none; removed FPGA_IO2_DAT, FPGA_IO2_DIR, FPGA_IO3_DAT, FPGA_IO3_DIR, JTAG_EN, TCK, TDI, TDO, TMS
- sheet mgt_refclk ports: added REFCLK_N, REFCLK_P; removed none
- sheet power ports: added none; removed 1V0_MGT, 1V2_MGT

Commit message: basic layout done
Connections:
- net IO_L1N_34: now reaches U21.1, U21.2
Changed lines of the file:
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@@
     )
   )
-  (global_label "IO_L9P_34" (shape bidirectional) (at 138.43 60.96 0) (fields_autoplaced)
-    (effects (font (size 1.27 1.27)) (justify left))
-    (property "Intersheetrefs" "${INTERSHEET_REFS}" (at 119.38 177.8 0)
+  (global_label "IO_L9P_34" (shape bidirectional) (at 43.18 177.8 0) (fields_autoplaced)
+    (effects (font (size 1.27 1.27)) (justify left))
+    (property "Intersheetrefs" "${INTERSHEET_REFS}" (at 24.13 60.96 0)
       (effects (font (size 1.27 1.27)) hide)
     )
@@
     )
   )
+  (global_label "IO_L18N_34" (shape bidirectional) (at 43.18 165.1 0) (fields_autoplaced)
+    (effects (font (size 1.27 1.27)) (justify left))
+    (property "Intersheetrefs" "${INTERSHEET_REFS}" (at 24.13 10.16 0)
+      (effects (font (size 1.27 1.27)) hide)
+    )
+  )
+  (global_label "IO_L16P_34" (shape bidirectional) (at 43.18 162.56 0) (fields_autoplaced)
+    (effects (font (size 1.27 1.27)) (justify left))
+    (property "Intersheetrefs" "${INTERSHEET_REFS}" (at 24.13 12.7 0)
+      (effects (font (size 1.27 1.27)) hide)
+    )
+  )
   (global_label "MGT_CLK0_P" (shape output) (at 44.45 59.69 0) (fields_autoplaced)
     (effects (font (size 1.27 1.27)) (justify left))
@@
     )
   )
+  (global_label "IO_L11N_34" (shape bidirectional) (at 236.22 160.02 0) (fields_autoplaced)
+    (effects (font (size 1.27 1.27)) (justify left))
+    (property "Intersheetrefs" "${INTERSHEET_REFS}" (at 250.4912 160.02 0)
+      (effects (font (size 1.27 1.27)) (justify left) hide)
+    )
+  )
   (global_label "IO_L11P_15" (shape bidirectional) (at 198.12 106.68 180) (fields_autoplaced)
     (effects (font (size 1.27 1.27)) (justify right))
@@
     )
   )
-  (global_label "IO_L9N_34" (shape bidirectional) (at 138.43 58.42 0) (fields_autoplaced)
-    (effects (font (size 1.27 1.27)) (justify left))
-    (property "Intersheetrefs" "${INTERSHEET_REFS}" (at 119.38 177.8 0)
+  (global_label "IO_L9N_34" (shape bidirectional) (at 43.18 180.34 0) (fields_autoplaced)
+    (effects (font (size 1.27 1.27)) (justify left))
+    (property "Intersheetrefs" "${INTERSHEET_REFS}" (at 24.13 60.96 0)
       (effects (font (size 1.27 1.27)) hide)
     )
@@
     )
   )
+  (global_label "IO_L24N_34" (shape bidirectional) (at 43.18 175.26 0) (fields_autoplaced)
+    (effects (font (size 1.27 1.27)) (justify left))
+    (property "Intersheetrefs" "${INTERSHEET_REFS}" (at 24.13 12.7 0)
+      (effects (font (size 1.27 1.27)) hide)
+    )
+  )
   (global_label "SCL0" (shape bidirectional) (at 132.08 68.58 180) (fields_autoplaced)
     (effects (font (size 1.27 1.27)) (justify right))
@@
     )
   )
+  (global_label "IO_L21P_34" (shape bidirectional) (at 236.22 154.94 0) (fields_autoplaced)
+    (effects (font (size 1.27 1.27)) (justify left))
+    (property "Intersheetrefs" "${INTERSHEET_REFS}" (at 250.4307 154.94 0)
+      (effects (font (size 1.27 1.27)) (justify left) hide)
+    )
+  )
+  (global_label "IO_L1N_34" (shape bidirectional) (at 139.7 48.26 0) (fields_autoplaced)
+    (effects (font (size 1.27 1.27)) (justify left))
+    (property "Intersheetrefs" "${INTERSHEET_REFS}" (at 152.7617 48.26 0)
+      (effects (font (size 1.27 1.27)) (justify left) hide)
+    )
+  )
   (global_label "IO_L6N_15" (shape bidirectional) (at 198.12 104.14 180) (fields_autoplaced)
     (effects (font (size 1.27 1.27)) (justify right))
@@
     )
   )
+  (global_label "IO_L3P_34" (shape bidirectional) (at 138.43 60.96 0) (fields_autoplaced)
+    (effects (font (size 1.27 1.27)) (justify left))
+    (property "Intersheetrefs" "${INTERSHEET_REFS}" (at 119.38 172.72 0)
+      (effects (font (size 1.27 1.27)) hide)
+    )
+  )
   (global_label "IO_L22N_15" (shape bidirectional) (at 198.12 124.46 180) (fields_autoplaced)
     (effects (font (size 1.27 1.27)) (justify right))
@@
     )
   )
+  (global_label "IO_L18P_34" (shape bidirectional) (at 43.18 170.18 0) (fields_autoplaced)
+    (effects (font (size 1.27 1.27)) (justify left))
+    (property "Intersheetrefs" "${INTERSHEET_REFS}" (at 24.13 17.78 0)
+      (effects (font (size 1.27 1.27)) hide)
+    )
+  )
   (global_label "IO_L13P_34" (shape bidirectional) (at 44.45 67.31 0) (fields_autoplaced)
     (effects (font (size 1.27 1.27)) (justify left))
@@
     )
   )
+  (global_label "IO_L20P_34" (shape bidirectional) (at 43.18 167.64 0) (fields_autoplaced)
+    (effects (font (size 1.27 1.27)) (justify left))
+    (property "Intersheetrefs" "${INTERSHEET_REFS}" (at 24.13 7.62 0)
+      (effects (font (size 1.27 1.27)) hide)
+    )
+  )
+  (global_label "IO_L14N_34" (shape bidirectional) (at 71.12 27.94 0) (fields_autoplaced)
+    (effects (font (size 1.27 1.27)) (justify left))
+    (property "Intersheetrefs" "${INTERSHEET_REFS}" (at 52.07 -109.22 0)
+      (effects (font (size 1.27 1.27)) hide)
+    )
+  )
   (global_label "IO_L23P_15" (shape bidirectional) (at 198.12 73.66 180) (fields_autoplaced)
     (effects (font (size 1.27 1.27)) (justify right))
@@
     )
   )
+  (global_label "IO_L19N_34" (shape bidirectional) (at 138.43 66.04 0) (fields_autoplaced)
+    (effects (font (size 1.27 1.27)) (justify left))
+    (property "Intersheetrefs" "${INTERSHEET_REFS}" (at 152.7012 66.04 0)
+      (effects (font (size 1.27 1.27)) (justify left) hide)
+    )
+  )
   (global_label "IO_L5P_15" (shape bidirectional) (at 198.12 81.28 180) (fields_autoplaced)
     (effects (font (size 1.27 1.27)) (justify right))
@@
     )
   )
+  (global_label "IO_L21N_34" (shape bidirectional) (at 138.43 68.58 0) (fields_autoplaced)
+    (effects (font (size 1.27 1.27)) (justify left))
+    (property "Intersheetrefs" "${INTERSHEET_REFS}" (at 152.7012 68.58 0)
+      (effects (font (size 1.27 1.27)) (justify left) hide)
+    )
+  )
   (global_label "IO_L9P_15" (shape bidirectional) (at 198.12 33.02 180) (fields_autoplaced)
     (effects (font (size 1.27 1.27)) (justify right))
@@
     )
   )
+  (global_label "IO_L1P_34" (shape bidirectional) (at 138.43 20.32 0) (fields_autoplaced)
+    (effects (font (size 1.27 1.27)) (justify left))
+    (property "Intersheetrefs" "${INTERSHEET_REFS}" (at 151.4312 20.32 0)
+      (effects (font (size 1.27 1.27)) (justify left) hide)
+    )
+  )
   (global_label "IO_L24N_15" (shape bidirectional) (at 198.12 58.42 180) (fields_autoplaced)
     (effects (font (size 1.27 1.27)) (justify right))
@@
     )
   )
+  (global_label "IO_L12N_34" (shape bidirectional) (at 236.22 151.13 0) (fields_autoplaced)
+    (effects (font (size 1.27 1.27)) (justify left))
+    (property "Intersheetrefs" "${INTERSHEET_REFS}" (at 250.4912 151.13 0)
+      (effects (font (size 1.27 1.27)) (justify left) hide)
+    )
+  )
   (global_label "IO_L7N_15" (shape bidirectional) (at 198.12 17.78 180) (fields_autoplaced)
     (effects (font (size 1.27 1.27)) (justify right))
@@
     )
   )
+  (global_label "IO_L2P_34" (shape bidirectional) (at 138.43 25.4 0) (fields_autoplaced)
+    (effects (font (size 1.27 1.27)) (justify left))
+    (property "Intersheetrefs" "${INTERSHEET_REFS}" (at 151.4312 25.4 0)
+      (effects (font (size 1.27 1.27)) (justify left) hide)
+    )
+  )
   (global_label "IO_L3N_15" (shape bidirectional) (at 198.12 78.74 180) (fields_autoplaced)
     (effects (font (size 1.27 1.27)) (justify right))
@@
     )
   )
+  (global_label "IO_L3N_34" (shape bidirectional) (at 138.43 58.42 0) (fields_autoplaced)
+    (effects (font (size 1.27 1.27)) (justify left))
+    (property "Intersheetrefs" "${INTERSHEET_REFS}" (at 119.38 172.72 0)
+      (effects (font (size 1.27 1.27)) hide)
+    )
+  )
+  (global_label "IO_L20N_34" (shape bidirectional) (at 43.18 172.72 0) (fields_autoplaced)
+    (effects (font (size 1.27 1.27)) (justify left))
+    (property "Intersheetrefs" "${INTERSHEET_REFS}" (at 24.13 15.24 0)
+      (effects (font (size 1.27 1.27)) hide)
+    )
+  )
   (global_label "IO_L16P_15" (shape bidirectional) (at 198.12 45.72 180) (fields_autoplaced)
     (effects (font (size 1.27 1.27)) (justify right))
@@
     )
   )
-  (global_label "IO_L20P_15" (shape bidirectional) (at 195.58 144.78 180) (fields_autoplaced)
-    (effects (font (size 1.27 1.27)) (justify right))
-    (property "Intersheetrefs" "${INTERSHEET_REFS}" (at 214.63 271.78 0)
-      (effects (font (size 1.27 1.27)) (justify left) hide)
+  (global_label "IO_L20P_15" (shape bidirectional) (at 236.22 157.48 0) (fields_autoplaced)
+    (effects (font (size 1.27 1.27)) (justify left))
+    (property "Intersheetrefs" "${INTERSHEET_REFS}" (at 250.4307 157.48 0)
+      (effects (font (size 1.27 1.27)) (justify left) hide)
+    )
+  )
+  (global_label "IO_L11P_34" (shape bidirectional) (at 195.58 144.78 180) (fields_autoplaced)
+    (effects (font (size 1.27 1.27)) (justify right))
+    (property "Intersheetrefs" "${INTERSHEET_REFS}" (at 214.63 12.7 0)
+      (effects (font (size 1.27 1.27)) hide)
     )
   )
@@
     )
   )
+  (global_label "IO_L19P_34" (shape bidirectional) (at 236.22 148.59 0) (fields_autoplaced)
+    (effects (font (size 1.27 1.27)) (justify left))
+    (property "Intersheetrefs" "${INTERSHEET_REFS}" (at 250.4307 148.59 0)
+      (effects (font (size 1.27 1.27)) (justify left) hide)
+    )
+  )
+  (global_label "IO_L2N_34" (shape bidirectional) (at 138.43 22.86 0) (fields_autoplaced)
+    (effects (font (size 1.27 1.27)) (justify left))
+    (property "Intersheetrefs" "${INTERSHEET_REFS}" (at 151.4917 22.86 0)
+      (effects (font (size 1.27 1.27)) (justify left) hide)
+    )
+  )
