File: kicad/leds.kicad_sch (KiCad schematic)
At the start: 21 parts, among them Q4 SSM6N35AFE, Q5 SSM6N35AFE, U14 74LVC1G06, U17 74LVC06

Commit message: WIP
Connections:
- net GND: now also Q5.4 (S); no longer Q5.1 (S)
- net LED7: now also Q5.5 (G); no longer Q5.2 (G)
- net LED_DONE_REF: now also Q4.5 (G); no longer Q4.2 (G)
- net LED_DONEb: now also Q4.4 (S); no longer Q4.1 (S)
- net at R10.2: now also Q5.3 (D); no longer Q5.6 (D)
- net at R99.2: now also Q4.3 (D); no longer Q4.6 (D)
