File: kicad/mgt_refclk.kicad_sch (KiCad schematic)
At the start: 23 parts, among them U12 5P49V6965, Y1 25MHz

Commit message: WIP
Parts:
- removed C90: 10u, Capacitor_SMD:C_1206_3216Metric, symbol Device:C_Small
- removed R67, R68: 50, Resistor_SMD:R_0603_1608Metric, symbol Device:R_Small
- removed R70, R71: 0, Resistor_SMD:R_0603_1608Metric, symbol Device:R_Small
Connections:
- net +1V8: now also C87.2, C89.1, U12.15 (VDDO3)
- net MGT_REFCLK_N renamed REFCLK_N
- net MGT_REFCLK_P renamed REFCLK_P
Other:
- note removed: "Only load 50Ohm HCSL termination resistors when not using LVDS."
- note removed: "Only load one bridge: LVDS -> 1V8 HCSL -> 3V3"
