File: kicad/peripherals_1.kicad_sch (KiCad schematic)
At the start: 26 parts, among them J4 JTAG, Q1 SSM6N35AFE, U3 FT240XQ, U8 74ALVC125

Commit message: WIP
Parts:
- removed C34, C35: 47p, Capacitor_SMD:C_0603_1608Metric, symbol Device:C_Small
- removed C36, C38, C39: 100n, Capacitor_SMD:C_0603_1608Metric, symbol fmc:100nF_603
- removed C37: 10u, Capacitor_SMD:C_1206_3216Metric, symbol Device:C_Small
- removed R19: 0, Resistor_SMD:R_0603_1608Metric, symbol Device:R_Small
- removed R20, R21: 27, Resistor_SMD:R_0603_1608Metric, symbol Device:R_Small
- removed U3: FT240XQ, Package_DFN_QFN:QFN-24-1EP_4x4mm_P0.5mm_EP2.6x2.6mm, symbol fmc:FT240XQ
Connections:
- net +1V8 renamed VREF_JTAG
- no-connect marks 1 -> 0
Other:
- moved on the sheet: R83
