File: kicad/power.kicad_sch (KiCad schematic)
At the start: 83 parts, among them J1 CUR_SEL, J2 PEN_SEL, J3 USB_C_Receptacle_USB2.0, Q2 SSM6N35AFE, Q3 Si3477, Q6 Si3477, Q7 SSM6N35AFE, U10 74LVC1G06, U11 UTC2000, U13 TPS3808DBV, U4 TLV62569ADDC, U5 TPS62A01A-SOT563, U6 TPS62A01A-SOT563, U7 TLV62569ADDC, U9 TLV62569ADDC

Commit message: WIP
Parts:
- removed C54, C55, C62, C63, C68: 10u, Capacitor_SMD:C_1206_3216Metric, symbol Device:C_Small
- removed C65, C66, C67, C75, C76: 22u, Capacitor_SMD:C_1206_3216Metric, symbol Device:C_Small
- removed C70, C71: 86p, Capacitor_SMD:C_0603_1608Metric, symbol Device:C_Small
- removed C72, C73: 56p, Capacitor_SMD:C_0603_1608Metric, symbol Device:C_Small
- removed C77: 100n, Capacitor_SMD:C_0603_1608Metric, symbol fmc:100nF_603
- removed J1: CUR_SEL, Connector_PinHeader_2.54mm:PinHeader_2x03_P2.54mm_Vertical, symbol Connector_Generic:Conn_02x03_Odd_Even
- removed J2: PEN_SEL, Connector_PinHeader_2.54mm:PinHeader_2x02_P2.54mm_Vertical, symbol Connector_Generic:Conn_02x02_Odd_Even
- removed L1, L6: 2u2, Inductor_SMD:L_Taiyo-Yuden_NR-50xx, symbol Device:L_Small
- removed L4, L5: 1u, Inductor_SMD:L_Taiyo-Yuden_NR-50xx, symbol Device:L_Small
- removed Q6: Si3477, Package_TO_SOT_SMD:TSOT-23-6, symbol fmc:Q_PMOS_DDGSDD
- removed Q7 (x2): SSM6N35AFE, proj_footprints:SOT-563-adjusted, symbol Device:Q_DUAL_NMOS_S1G1D2S2G2D1
- removed R22, R23, R24, R25: 100k, Resistor_SMD:R_0603_1608Metric, symbol Device:R_Small
- removed R34, R46, R47, R48, R49, R50: 0, Resistor_SMD:R_0603_1608Metric, symbol Device:R_Small
- removed R35, R52, R54, R55, R58, R59: 10k, Resistor_SMD:R_0603_1608Metric, symbol Device:R_Small
- removed R36, R37, R38, R43, R44: 24k, Resistor_SMD:R_0603_1608Metric, symbol Device:R_Small
- removed R39: 12k, Resistor_SMD:R_0603_1608Metric, symbol Device:R_Small
- removed R41, R42: 16k, Resistor_SMD:R_0603_1608Metric, symbol Device:R_Small
- removed R60: 5k1, Resistor_SMD:R_0603_1608Metric, symbol Device:R_Small
- removed R61: 35k7, Resistor_SMD:R_0603_1608Metric, symbol Device:R_Small
- removed TP14: TestPoint, TestPoint:TestPoint_Pad_D1.0mm, symbol Connector:TestPoint
- removed U11: UTC2000, Package_DFN_QFN:QFN-16-1EP_3x3mm_P0.5mm_EP1.75x1.75mm_ThermalVias, symbol fmc:UTC2000
- removed U4, U7: TLV62569ADDC, Package_TO_SOT_SMD:SOT-23-6, symbol Regulator_Switching:TLV62569DDC
- removed U5, U6: TPS62A01A-SOT563, Package_TO_SOT_SMD:SOT-563, symbol fmc:TPS62A01-SOT563
- added JP1: 3V3, Connector_PinHeader_2.54mm:PinHeader_1x02_P2.54mm_Vertical, symbol Jumper:Jumper_2_Bridged
- added JP2: PWR, Connector_PinHeader_2.54mm:PinHeader_1x02_P2.54mm_Vertical, symbol Jumper:Jumper_2_Bridged
- added TP2306: GND, Connector_PinHeader_2.54mm:PinHeader_1x01_P2.54mm_Vertical, symbol Connector:TestPoint
- J3: footprint proj_footprints:USB_C_Receptacle_GCT_USB4085_smaller_holes -> Connector_USB:USB_C_Receptacle_JAE_DX07S016JA1R1500
Connections:
- net +3V3: now also JP1.2 (B); no longer C74.1, R45.1
- net GND: now also Q2.4 (S), JP2.2 (B); no longer Q2.1 (S)
- net POWER_CYCLE: now also Q2.5 (G); no longer Q2.2 (G)
- net PWR_EN: now also R33.1, U9.1 (EN)
- net at R53.2, U10.1, U10.2: now also JP2.1 (A)
- net at U13.3 (~{MR}): now also Q2.3 (D); no longer Q2.6 (D)
- net at C69.1, L7.2: now also C74.1, R45.1, JP1.1 (A)
- net USBin_N: no longer names the net of J3.A7 (D-)
- net USBin_N: no longer J3.B7 (D-)
- net USBin_P: no longer names the net of J3.A6 (D+)
- net USBin_P: no longer J3.B6 (D+)
- new net GND_lan9254: TP2306.1
Other:
- note removed: "Use forced-PWM regulator for reduced ripple!"
