File: kicad/no_conn.kicad_sch (KiCad schematic)
At the start: 10 parts

Commit message: WIP
Parts:
- removed TP1, TP10, TP11, TP12, TP13, TP2, TP3, TP4, TP6, TP7: Dummy End, proj_footprints:endpoint_0.1mm, symbol Connector:TestPoint_Small
Connections:
- no-connect marks 42 -> 0
Other:
- note removed: "AUX ADC"
- note removed: "Testpoints on this page are pins that are currently unused but have been routed to the edge of the FPGA."

Commit message: basic layout done
Connections:
- no-connect marks 0 -> 83

Commit message: further work; will need to redo vias :-( for jlcpcb
Connections:
- no-connect marks 83 -> 79
Changed lines of the file:
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@@
   (no_connect (at 146.05 109.22))
   (no_connect (at 146.05 106.68))
-  (no_connect (at 72.39 130.81))
   (no_connect (at 167.64 129.54))
   (no_connect (at 167.64 142.24))
@@
   (no_connect (at 146.05 147.32))
   (no_connect (at 72.39 133.35))
-  (no_connect (at 72.39 59.69))
   (no_connect (at 167.64 109.22))
   (no_connect (at 167.64 132.08))
@@
   (no_connect (at 54.61 146.05))
   (no_connect (at 54.61 46.99))
-  (no_connect (at 72.39 67.31))
   (no_connect (at 146.05 142.24))
   (no_connect (at 167.64 147.32))
@@
   (no_connect (at 72.39 46.99))
   (no_connect (at 146.05 104.14))
-  (no_connect (at 72.39 52.07))
   (no_connect (at 72.39 69.85))
   (no_connect (at 72.39 77.47))
